File: drsstc.sch (EAGLE design)
At the start: 122 parts, among them U1 AP1501, U10 LM311, U11 74HC74, U12 LM8365, U13 ICM7216D, U14 ICM7216D, U2 74AHCT1G32, U3 AP1506, U4 MCP4706, U5 UCC27423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

Commit message: Updating DRSSTC board to Rev B
Parts:
- removed CNTRL: (no value), pinhead:PINHD-1X6
- added MODE, MSTR, TEST, TRIG: (no value), pinhead:PINHD-1X2
- R15: device resistor:R-US_R1206 -> drsstc:51OHM_RES
- TP2: device pinhead:PINHD-1X4 -> pinhead:PINHD-1X6
Connections:
- removed net MODE1: CNTRL.3, JP5.A2, R2.1
- removed net MODE2: CNTRL.4, JP5.A1, R3.1
- removed net N$26: D4.C, D5.A, R14.1, TP2.1, U6.-IN
- removed net POT: CNTRL.2, JP5.A3, R1.1
- new net FB_IN: D4.C, D5.A, R14.1, TP2.2, U6.-IN
- new net MODE: JP5.A1, MODE.1, R3.1
- new net TEST: JP5.A2, R2.1, TEST.1
- new net TRIG: JP5.A3, R1.1, TRIG.1
- net ACTIVE: now also TP2.6
- net GND: now also NEOPIXEL.3, TP2.1, U2.GND, U6.LATCH_EN; no longer CNTRL.1, NEOPIXEL.2, TP2.2, U2.VCC, U6.VCC+
- net INA: now also TP2.5
- net MSTR_EN: now also MSTR.1; no longer CNTRL.5
- net N$13: now also NEOPIXEL.2; no longer NEOPIXEL.3
- net VCC: now also MODE.2, MSTR.2, TEST.2, TRIG.2, U2.VCC, U6.VCC+; no longer CNTRL.6, U2.GND, U6.LATCH_EN
Other:
- moved on the sheet: C1

Commit message: Updating Rev B board, linking freq counter to driver input signal
Connections:
- net INA: now also U14.INPUT_A
- net PRIMARY: no longer U14.INPUT_A
Changed lines of the file:
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@@
 <setting verticaltext="up"/>
 </settings>
-<grid distance="0.05" unitdist="inch" unit="inch" style="lines" multiple="1" display="no" altdistance="0.01" altunitdist="inch" altunit="inch"/>
+<grid distance="0.1" unitdist="inch" unit="inch" style="lines" multiple="1" display="no" altdistance="0.01" altunitdist="inch" altunit="inch"/>
 <layers>
 <layer number="1" name="Top" color="4" fill="1" visible="no" active="no"/>
@@
 <net name="PRIMARY" class="0">
 <segment>
-<pinref part="U14" gate="G$1" pin="INPUT_A"/>
-<wire x1="-74.93" y1="82.55" x2="-102.87" y2="82.55" width="0.1524" layer="91"/>
-<label x="-102.87" y="82.55" size="1.778" layer="95" rot="R180" xref="yes"/>
-</segment>
-<segment>
 <wire x1="-85.09" y1="203.2" x2="-85.09" y2="210.82" width="0.1524" layer="91"/>
 <wire x1="-85.09" y1="210.82" x2="-85.09" y2="213.36" width="0.1524" layer="91"/>
@@
 <wire x1="-13.97" y1="219.71" x2="-13.97" y2="209.55" width="0.1524" layer="91"/>
 </segment>
-</net>
+<segment>
+<pinref part="U14" gate="G$1" pin="INPUT_A"/>
+<wire x1="-74.93" y1="82.55" x2="-102.87" y2="82.55" width="0.1524" layer="91"/>
+<label x="-102.87" y="82.55" size="1.778" layer="95" rot="R180" xref="yes"/>
+</segment>
+</net>

Commit message: Updating Rev B board with hysteresis feedback fix
Connections:
- new net N$26: R13.1, R17.2, U6.+IN
- net FB_IN: now also R10.2, R8.2
- net INA: now also U7.INB; no longer U7.INA
- net INB: now also U7.INA; no longer U7.INB
- net N$23: now also C9.2, R10.1, U6./Q; no longer R10.2, R13.1, R17.2, R8.2, U6.+IN
- net PRIMARY: no longer C9.2, R10.1
Other:
- moved on the sheet: C14
